File: PCB/mp3_player/mp3_player.kicad_pcb (KiCad board)
At the start: 2 copper layers, 33 parts, among them J1 FRDM-K64F, J2 Conn_01x03_Pin, J3 Conn_01x04_Pin, J4 Terminal_2, J5 Conn_01x02_Pin, J6 Connector_3, J7 Conn_01x02_Pin, Q1 TIP32, Q2 TIP31, SW1 RotaryEncoder_Switch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

Commit message: feat: PCB ready
Parts:
- removed J5: Conn_01x02_Pin, Connector_PinSocket_2.54mm:PinSocket_1x02_P2.54mm_Vertical
- removed J6: Connector_3, TCLib:PinHeader_1x03_P2.54mm_Vertical
- added JP1: Jumper_2_Bridged, TestPoint:TestPoint_2Pads_Pitch2.54mm_Drill0.8mm, F.Cu at (209.5, 136.5)
- J2: footprint Connector_PinHeader_2.54mm:PinHeader_1x03_P2.54mm_Horizontal -> Connector_PinHeader_2.54mm:PinHeader_1x03_P2.54mm_Vertical
- J7: value Conn_01x02_Pin -> Connector_2_Pol; footprint Connector_PinSocket_2.54mm:PinSocket_1x02_P2.54mm_Vertical -> TCLib:Molex_1x02_P2.54mm
- U1: footprint Package_TO_SOT_THT:TO-220-3_Vertical -> Package_TO_SOT_THT:TO-220-3_Horizontal_TabDown
- moved J1 187.1 mm to (172.1, 77.2)
- moved R10 102.4 mm to (222.3, 125.8)
- moved C6 97.8 mm to (214.0, 104.3), turned to 180 degrees
- moved C7 97.8 mm to (214.0, 114.8), turned to 180 degrees
- moved D1 95.5 mm to (224.0, 108.6), turned to 90 degrees
- moved D2 95.4 mm to (224.0, 120.1), turned to 90 degrees
- moved R3 93.7 mm to (138.6, 89.5), turned to 180 degrees
- moved R4 93.0 mm to (138.7, 84.0), turned to 180 degrees
- moved Q1 89.7 mm to (232.0, 114.2), turned to -90 degrees
- moved Q2 89.4 mm to (232.0, 101.2), turned to -90 degrees
- moved R11 85.3 mm to (234.1, 95.8), turned to 180 degrees
- moved R5 81.5 mm to (177.8, 137.8), turned to 180 degrees
- moved C5 73.1 mm to (243.5, 122.0), turned to -90 degrees
- moved S1 72.8 mm to (173.1, 129.5)
- moved S2 71.7 mm to (190.6, 129.5)
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Connections:
- J1 pad J1-11: /enc_RCHA -> unconnected-(J1-PTC0-PadJ1-11)
- J1 pad J1-6: /bt_prev -> unconnected-(J1-PTB9-PadJ1-6)
- J1 pad J1-7: /enc_sw -> /enc_RCHB
- J1 pad J1-9: /enc_RCHB -> /enc_RCHA
- J1 pad J2-5: unconnected-(J1-ADC0_DP0-PadJ2-5) -> /enc_sw
- J1 pad J2-7: unconnected-(J1-ADC0_DM0-PadJ2-7) -> /bt_prev
- J1 pad J4-2: /bt_play/stop -> unconnected-(J1-PTB2-PadJ4-2)
- J1 pad J4-4: /bt_next -> unconnected-(J1-PTB3-PadJ4-4)
- J1 pad J4-7: unconnected-(J1-ADC1_DM1-PadJ4-7) -> /bt_play/stop
- J1 pad J4-9: unconnected-(J1-PTB20-PadJ4-9) -> /bt_next
- J7 pad 1: /etapa_salida -> GND
- J7 pad 2: GND -> /etapa_salida
Routing:
- net GND: track 0.00 -> 678.5 mm
- net +3V3: track 0.00 -> 240.6 mm, vias 0 -> 1
- net +5V: track 0.00 -> 232.1 mm, vias 0 -> 2
- net /sda: track 0.00 -> 120.3 mm
- net /scl: track 0.00 -> 108.3 mm
- net /matriz_led: track 0.00 -> 100.4 mm
- net /enc_sw: track 0.00 -> 83.7 mm
- net +12V: track 0.00 -> 73.7 mm
- net /bt_prev: track 0.00 -> 73.3 mm
- net /DAC_out: track 0.00 -> 68.9 mm
- net /bt_play/stop: track 0.00 -> 51.3 mm
- net /etapa_salida: track 0.00 -> 42.6 mm
- net /bt_next: track 0.00 -> 42.4 mm
- net /enc_RCHA: track 0.00 -> 42.1 mm
- net /enc_RCHB: track 0.00 -> 41.4 mm
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Other:
- board outline added: 200 x 100 mm
- board text added: "+12V"
- board text added: "GND"
- board text added: "OUTPUT STAGE"
- board text added: "Vo"
- board text added: "bypass output stage"
