File: PCB/mp3_player/mp3_player.kicad_sch (KiCad schematic)
At the start: 0 parts

Commit message: feat: esquematico listo para revisar
Parts:
- added C1, C2: C, TCLib:C_5mm, symbol TCLib:C
- added C3, C4, C5, C6, C7: C_Polarized, TCLib:CP_2.50mm, symbol TCLib:C_Polarized
- added D1, D2: 1N4148, Diode_THT:D_DO-35_SOD27_P7.62mm_Horizontal, symbol Diode:1N4148
- added J1: FRDM-K64F, SistEmb:FRDM-K64F, symbol SistEmb:FRDM-K64F
- added J2: Conn_01x03_Pin, Connector_PinHeader_2.54mm:PinHeader_1x03_P2.54mm_Horizontal, symbol Connector:Conn_01x03_Pin
- added J3: Conn_01x04_Pin, Connector_PinHeader_2.54mm:PinHeader_1x04_P2.54mm_Vertical, symbol Connector:Conn_01x04_Pin
- added J4: Terminal_2, TCLib:Bornera_2_P5mm, symbol TCLib:Terminal_2
- added J5, J7: Conn_01x02_Pin, Connector_PinSocket_2.54mm:PinSocket_1x02_P2.54mm_Vertical, symbol Connector:Conn_01x02_Pin
- added J6: Connector_3, TCLib:PinHeader_1x03_P2.54mm_Vertical, symbol TCLib:Connector_3
- added Q1: TIP32, TCLib:TO-220-3_Vertical, symbol TCLib:TIP32
- added Q2: TIP31, TCLib:TO-220-3_Vertical, symbol TCLib:TIP31
- added R1, R2: 10k, TCLib:R_0.25W, symbol TCLib:R
- added R10, R11, R3, R4: R, TCLib:R_0.25W, symbol TCLib:R
- added R5, R6, R7, R8: 1k, TCLib:R_0.25W, symbol TCLib:R
- added S1, S2, S3: SW_Tactile, TCLib:SW_Tactile, symbol TCLib:SW_Tactile
- added SW1: RotaryEncoder_Switch, SistEmb:XDCR_PEC12R-4115F-S0012, symbol Device:RotaryEncoder_Switch
- added U1: L7805, Package_TO_SOT_THT:TO-220-3_Vertical, symbol Regulator_Linear:L7805
Connections:
- new net: C6.1, D1.2 (A), Q2.1 (B), R11.2
- new net: D1.1 (K), D2.2 (A)
- new net: C7.1, D2.1 (K), Q1.1 (B), R10.1
- new net: J5.1 (Pin_1), J6.2
- new net: C5.1, Q1.3 (E), Q2.3 (E)
- new net +12V: C2.1, C4.1, J4.2, Q2.2 (C), R11.1, U1.1 (IN)
- new net +3V3: J1.J3-4 (P3V3_1), J1.J3-8 (P3V3_2), R1.1, R2.2, R3.1, R4.1, S1.1, S1.2, S2.1, S2.2, S3.1, S3.2, SW1.S2
- new net +5V: C1.1, C3.1, J1.J3-16 (P5-9V_VIN), J2.2 (Pin_2), J3.3 (Pin_3), U1.3 (OUT)
- new net DAC_out: C6.2, C7.2, J1.J4-11 (DAC0_OUT), J6.3
- new net GND: C1.2, C2.2, C3.2, C4.2, J1.J2-14 (GND1), J1.J2-3 (GND0), J1.J3-12 (GND2), J1.J3-14 (GND3), J2.3 (Pin_3), J3.4 (Pin_4), J4.1, J5.2 (Pin_2), J7.2 (Pin_2), Q1.2 (C), R10.2, R5.2, R6.2, R7.2, R8.2, SW1.C, U1.2 (GND)
- new net bt_next: J1.J4-4 (PTB3), R6.1, S2.3, S2.4
- new net bt_play/stop: J1.J4-2 (PTB2), R5.1, S1.3, S1.4
- new net bt_prev: J1.J1-6 (PTB9), R7.1, S3.3, S3.4
- new net enc_RCHA: J1.J1-11 (PTC0), R2.1, SW1.A
- new net enc_RCHB: J1.J1-9 (PTC9), R1.2, SW1.B
- new net enc_sw: J1.J1-7 (PTC8), R8.1, SW1.S1
- new net etapa_salida: C5.2, J6.1, J7.1 (Pin_1)
- new net matriz_led: J1.J1-5 (PTC1), J2.1 (Pin_1)
- new net scl: J1.J2-20 (PTE24), J3.1 (Pin_1), R4.2
- new net sda: J1.J2-18 (PTE25), J3.2 (Pin_2), R3.2
Other:
- note added: "ALIMENTACION"
- note added: "BOTONES"
- note added: "DISPLAY LCD"
- note added: "ENCODER"
- note added: "ETAPA SALIDA"
- note added: "MATRIZ LED"
- note added: "SALIDA AUDIO"

Commit message: feat: PCB ready
Parts:
- removed J5, J7: Conn_01x02_Pin, Connector_PinSocket_2.54mm:PinSocket_1x02_P2.54mm_Vertical, symbol Connector:Conn_01x02_Pin
- removed J6: Connector_3, TCLib:PinHeader_1x03_P2.54mm_Vertical, symbol TCLib:Connector_3
- added J7: Connector_2_Pol, TCLib:Molex_1x02_P2.54mm, symbol TCLib:Connector_2_Pol
- added JP1: Jumper_2_Bridged, TestPoint:TestPoint_2Pads_Pitch2.54mm_Drill0.8mm, symbol Jumper:Jumper_2_Bridged
- J2: footprint Connector_PinHeader_2.54mm:PinHeader_1x03_P2.54mm_Horizontal -> Connector_PinHeader_2.54mm:PinHeader_1x03_P2.54mm_Vertical
- U1: footprint Package_TO_SOT_THT:TO-220-3_Vertical -> Package_TO_SOT_THT:TO-220-3_Horizontal_TabDown
Connections:
- net +12V: now also J4.1; no longer J4.2
- net DAC_out: now also JP1.1 (A)
- net GND: now also J4.2, J7.1; no longer J4.1
- net bt_next: now also J1.J4-9 (PTB20); no longer J1.J4-4 (PTB3)
- net bt_play/stop: now also J1.J4-7 (ADC1_DM1); no longer J1.J4-2 (PTB2)
- net bt_prev: now also J1.J2-7 (ADC0_DM0); no longer J1.J1-6 (PTB9)
- net enc_RCHA: now also J1.J1-9 (PTC9); no longer J1.J1-11 (PTC0)
- net enc_RCHB: now also J1.J1-7 (PTC8); no longer J1.J1-9 (PTC9)
- net enc_sw: now also J1.J2-5 (ADC0_DP0); no longer J1.J1-7 (PTC8)
- net etapa_salida: now also J7.2, JP1.2 (B)
Other:
- moved on the sheet: R2
